File: ECAD/NinjaPAMI-2026/NinjaPAMI-2026.kicad_sch (KiCad schematic)
At the start: 42 parts, among them J1 Sensor_Center, J11 Con_Batt, J13 OLED, J2 Conn_01x04, J3 Sensor_RIGHT, J4 Servo, J5 Sensor_LEFT, J6 Servo, J7 LeftMotor, J8 RightMotor, SW1 SW_SPDT, SW2 SW_Reed, SW3 SW_SPDT, U1 XIAO-HALF-HOLE-23P, U3 TMC2208_SILENTSTEPSTICK, U4 TMC2208_SILENTSTEPSTICK, U5 R-78E5.0-1.0

Commit message: PAMI ninja PCB update
Parts:
- removed U3, U4: TMC2208_SILENTSTEPSTICK, PAMI-2025:Step-Stick Driver Bottom Entry Version, symbol PAMI-2025:TMC2208_SILENTSTEPSTICK
- added D10, D11, D3, D6: LED_Small, LED_SMD:LED_1206_3216Metric_Pad1.42x1.75mm_HandSolder, symbol Device:LED_Small
- added D13, D14, D4, D7: D_Small, Diode_SMD:D_SMA_Handsoldering, symbol Device:D_Small
- added J10: CON_EV_01, Connector_Molex:Molex_KK-254_AE-6410-02A_1x02_P2.54mm_Vertical, symbol Connector_Generic:Conn_01x02
- added J7, J8: CON_EV_02, Connector_Molex:Molex_KK-254_AE-6410-02A_1x02_P2.54mm_Vertical, symbol Connector_Generic:Conn_01x02
- added J9: CON_PUMP_01, Connector_Molex:Molex_KK-254_AE-6410-02A_1x02_P2.54mm_Vertical, symbol Connector_Generic:Conn_01x02
- added JP1, JP2, JP3, JP4, JP5, JP6: SolderJumper_3_Open, Jumper:SolderJumper-3_P1.3mm_Open_RoundedPad1.0x1.5mm_NumberLabels, symbol Jumper:SolderJumper_3_Open
- added Q1, Q2, Q3, Q4: AO3400A, Package_TO_SOT_SMD:SOT-23, symbol Transistor_FET:AO3400A
- added R10, R13, R19, R20: 270R, Resistor_SMD:R_1206_3216Metric_Pad1.30x1.75mm_HandSolder, symbol Device:R_Small
- added R11, R14, R21, R22: 10K, Resistor_SMD:R_1206_3216Metric_Pad1.30x1.75mm_HandSolder, symbol Device:R_Small
- added R12, R17, R18, R9: 1K, Resistor_SMD:R_1206_3216Metric_Pad1.30x1.75mm_HandSolder, symbol Device:R_Small
- added U3, U4: TMC2209_SILENTSTEPSTICK, TMC2209_SILENTSTEPSTICK:MODULE_TMC2209_SILENTSTEPSTICK, symbol TMC2209_SILENTSTEPSTICK:TMC2209_SILENTSTEPSTICK
- J13: renamed from J8; footprint Connector_PinHeader_2.54mm:PinHeader_1x04_P2.54mm_Vertical -> Connector_Molex:Molex_KK-254_AE-6410-04A_1x04_P2.54mm_Vertical
- J14: renamed from J7; footprint Connector_PinHeader_2.54mm:PinHeader_1x04_P2.54mm_Vertical -> Connector_Molex:Molex_KK-254_AE-6410-04A_1x04_P2.54mm_Vertical
- J4: renamed from J3; footprint PAMI-2025:VL53 Bottom Entry Version -> Connector_Molex:Molex_KK-254_AE-6410-06A_1x06_P2.54mm_Vertical
- J5: renamed from J1; footprint PAMI-2025:VL53 Bottom Entry Version -> Connector_Molex:Molex_KK-254_AE-6410-06A_1x06_P2.54mm_Vertical
- J6: renamed from J5; footprint PAMI-2025:VL53 Bottom Entry Version -> Connector_Molex:Molex_KK-254_AE-6410-06A_1x06_P2.54mm_Vertical
- renumbered BZ2 to BZ1, C10 to C1, C11 to C2, C7 to C3, C6 to C4, D3 to D12, D4 to D2, D2 to D5, D10 to D8, D5 to D9, J11 to J1, J2 to J11, J13 to J12, J4 to J2, J6 to J3, R7 to R1, R13 to R15, R4 to R16, R10 to R2, R8 to R3, R11 to R4, R6 to R5, R12 to R6, R3 to R7, R2 to R8, SW3 to SW1, SW1 to SW3, U5 to U1, U1 to U2
Connections:
- net +3.3V: now also U3.2 (VIO), U4.2 (VIO)
- net +9V: now also JP2.1 (A), JP3.1 (A), JP5.1 (A), JP6.1 (A), U3.8 (VM), U4.8 (VM)
- net EnDriver: now also U3.16 (~{EN}), U4.16 (~{EN})
- net GND: now also D10.1 (K), D11.1 (K), D3.1 (K), D6.1 (K), Q1.2 (S), Q2.2 (S), Q3.2 (S), Q4.2 (S), R11.2, R14.2, R21.2, R22.2, U3.1 (GND), U3.7 (GND), U4.1 (GND), U4.7 (GND)
- net LeftDir: now also U4.10 (STEP)
- net LeftMS1: now also U3.15 (MS1), U4.15 (MS1)
- net LeftMS2: now also U3.14 (MS2), U4.14 (MS2)
- net LeftStep: now also U4.9 (DIR)
- net RX: now also JP4.1 (A); no longer U2.8 (U0RXD_D7/RX)
- net RightDir: now also U3.10 (STEP)
- net RightStep: now also U3.9 (DIR)
- net TX: now also JP1.3 (B); no longer U2.7 (U0TXD_D6/TX)
- net XSHUT_LEFT: now also JP4.3 (B)
- net XSHUT_RIGHT: now also JP1.1 (A)
- net at J14.1 (Pin_1): now also U4.3 (M1B)
- net at J14.2 (Pin_2): now also U4.4 (M1A)
- net at J14.3 (Pin_3): now also U4.5 (M2A)
- net at J14.4 (Pin_4): now also U4.6 (M2B)
- net at J13.1 (Pin_1): now also U3.3 (M1B)
- net at J13.2 (Pin_2): now also U3.4 (M1A)
- net at J13.3 (Pin_3): now also U3.5 (M2A)
- net at J13.4 (Pin_4): now also U3.6 (M2B)
- new net: JP4.2 (C), U2.8 (U0RXD_D7/RX)
- new net: Q1.1 (G), R10.1, R11.1
- new net: D10.2 (A), R17.2
- new net: Q2.1 (G), R13.1, R14.1
- new net: D14.1 (K), J10.2 (Pin_2), JP6.2 (C)
- new net: D13.1 (K), J9.2 (Pin_2), JP5.2 (C)
- new net: D11.2 (A), R18.2
- new net: Q4.1 (G), R20.1, R22.1
- new net: D14.2 (A), J10.1 (Pin_1), Q4.3 (D)
- new net: D6.2 (A), R12.2
- new net: Q3.1 (G), R19.1, R21.1
- new net: D7.1 (K), J8.2 (Pin_2), JP3.2 (C)
- new net: D7.2 (A), J8.1 (Pin_1), Q2.3 (D)
- new net: JP1.2 (C), U2.7 (U0TXD_D6/TX)
- new net: D3.2 (A), R9.2
- new net: D4.2 (A), J7.1 (Pin_1), Q1.3 (D)
- new net: D4.1 (K), J7.2 (Pin_2), JP2.2 (C)
- new net: D13.2 (A), J9.1 (Pin_1), Q3.3 (D)
- new net +5V: JP2.3 (B), JP3.3 (B), JP5.3 (B), JP6.3 (B)
- new net S_EV_01: R18.1, R20.2
- new net S_EV_02: R12.1, R13.2
- new net S_PUMP_01: R17.1, R19.2
- new net S_PUMP_02: R10.2, R9.1
- no-connect marks 7 -> 9
Other:
- moved on the sheet: BZ1, J12, J2, J3, R1, R2, R3, R4, R5, R6, SW2, SW3
